Commit message: feat: real-robot bringup — URDF align + EKF config + teleop stop suppression + calibration tools
Real-robot bringup tightened after physical testing on the SMB chassis.

smb_robot/urdf/smb.urdf.xacro
  - Wheels at FRONT (x=+0.05), caster at BACK (x=-0.05). The previous
    layout had it inverted.
  - Lidar moved to LEFT side (x=-0.05) and rotated -90° about Z so
    angle_min=0 points along URDF +Y (physical forward, wall side).
  - Adds explicit convention comment: URDF +X = arrow/ESP32 motor
    direction = physical forward; odom +X = URDF +X (no flip).

smb_robot_bringup/config/robot/ekf_minimal.yaml
  - /odom_relay now publishes yaw_rate as well (the angular.z
    component). The EKF was rejecting heading changes because the
    config masked the third row. Toggling false→true on the
    yaw_rate column lets the filter fuse gyro-corrected odometry.

smb_robot_bringup/config/robot/slam_toolbox.yaml
  - scan_queue_size 5 → 20 so 1-2 Hz ESP32 scans don't get dropped.
  - transform_tolerance 0.25 → 0.5 s: with 1 Hz scans the
    scan-to-pose transform can lag, and the smaller value was
    rejecting valid matches.

smb_nodes/smb_nodes/supervisor.py
  - Stop suppression: when teleop sends lin=0 (key released) the
    supervisor stops publishing /cmd_vel entirely. The ESP32's own
    500 ms watchdog handles stopping the wheels. Without this
    branch the supervisor flooded /cmd_vel with zeros at 10 Hz
    between teleop key presses, triggering botStop() on every
    republish tick and producing micro-step jitter.

test_robot.sh
  - Adds --no-nav2 flag: use_nav2:=false use_slam:=false for
    teleop-only bringup. SLAM scan-matching fails when the
    robot is moved outside the scanned area, so map→odom drifts
    and Nav2 fights teleop.
  - auto_activate probes ros2 node list before invoking SLAM
    and Nav2 lifecycle ops so the script no longer hard-exits
    when those components are absent.

test_calibration.sh, test_odom_drift.sh
  - WHEEL_DIAM_M and WHEEL_BASE_M calibration helpers. These
    measure actual hardware dimensions and produce corrected
    Config.h values for ESP32 firmware. See top-of-file
    comments for the workflow.

Co-authored-by: Cursor <cursoragent@cursor.com>

File: src/smb_robot/urdf/smb.urdf.xacro (robot description, xacro)
@@ -21,10 +21,12 @@
   <xacro:property name="wheel_thickness" value="0.02"/>
   <xacro:property name="track"          value="0.22"/>
-  <!-- Drive wheels at the REAR of the chassis (x = -0.05), driven by motors with
-       encoders — matches the real robot layout. Single ball caster at the front
-       (x = +0.05) for free-rolling turns. Ball joint is critical: the front caster
-       must roll freely during rotation so DiffDrive odometry stays accurate. -->
-  <xacro:property name="wheel_offset_x" value="-0.05"/>
-  <xacro:property name="caster_offset_x" value="+0.05"/>
+  <!-- Drive wheels at the FRONT of the chassis (x = +0.05) — driven by motors with
+       encoders. Single ball caster at the BACK (x = -0.05) for free-rolling turns.
+       Convention: URDF +X = physical forward = arrow/ESP32 side = motor direction.
+       ESP32 odom +X = motor direction = URDF +X. No odom flip needed.
+       Scan data: lidar on back (-X) with 180° rotation so angle 0° faces backward
+       (toward wall = physical front). -->
+  <xacro:property name="wheel_offset_x" value="0.05"/>
+  <xacro:property name="caster_offset_x" value="-0.05"/>
   <!-- Caster uses the same radius as the drive wheels so all three contact
        points lie on the same ground plane. The wheel_radius property above
@@ -174,9 +176,13 @@
     </collision>
   </link>
-  <!-- Laser frame: top of chassis, +z by lidar_offset_z. Yaw = 0 (forward-facing). -->
+  <!-- Laser frame: mounted on the LEFT side of chassis (x = -0.05, y = 0),
+       with -90° yaw so lidar angle_min=0 points along URDF +Y = physical forward (wall).
+       Scan data: wall at ~315-340° = URDF +Y direction. ESP32 publishes angle 0°
+       in the chassis +Y direction, so rpy=0 0 -1.5708 makes lidar +X align with chassis +Y. -->
+  <xacro:property name="lidar_offset_x" value="-0.05"/>
   <joint name="lidar_joint" type="fixed">
     <parent link="base_link"/>
     <child link="laser_frame"/>
-    <origin xyz="0 0 ${lidar_offset_z}" rpy="0 0 0"/>
+    <origin xyz="${lidar_offset_x} 0 ${lidar_offset_z}" rpy="0 0 -1.5707"/>
   </joint>
   <link name="laser_frame">
