Commit message: fix: Fix robot simulation

File: src/smb_robot/urdf/smb.urdf.xacro (robot description, xacro)
@@ -21,11 +21,19 @@
   <xacro:property name="wheel_thickness" value="0.02"/>
   <xacro:property name="track"          value="0.22"/>
-  <xacro:property name="caster_offset_x" value="-0.13"/>
-  <xacro:property name="caster_radius"  value="0.02"/>
+  <!-- Drive wheels forward of chassis center (x = +0.05), single caster at the
+       rear (x = -0.105). This mirrors the visualize_lidar.sdf reference layout:
+       wheels carry the front load, caster balances the rear. Masses/inertia
+       sized for a chibi ~30cm supermarket robot. -->
+  <xacro:property name="wheel_offset_x" value="0.05"/>
+  <xacro:property name="caster_offset_x" value="-0.105"/>
+  <!-- Caster uses the same radius as the drive wheels so all three contact
+       points lie on the same ground plane. The wheel_radius property above
+       is reused for the caster sphere. -->
   <xacro:property name="lidar_offset_z" value="0.075"/>
   <xacro:property name="imu_offset_z"   value="0.05"/>
-  <xacro:property name="chassis_mass"   value="1.14395"/>
-  <xacro:property name="wheel_mass"     value="2.0"/>
-  <xacro:property name="caster_mass"    value="1.0"/>
+  <!-- Masses kept low so the sim runs smoothly; chassis dominates the dynamics. -->
+  <xacro:property name="chassis_mass"   value="2.0"/>
+  <xacro:property name="wheel_mass"     value="0.1"/>
+  <xacro:property name="caster_mass"    value="0.05"/>
   <link name="base_link">
     <!-- KDL doesn't support a root link with inertia, but RobotDescription does.
@@ -36,8 +44,12 @@
       <origin xyz="0 0 0" rpy="0 0 0"/>
       <mass value="${chassis_mass}"/>
-      <inertia
-        ixx="0.126164" ixy="0" ixz="0"
-        iyy="0.416519" iyz="0"
-        izz="0.481014"/>
+      <!-- Box inertia for 0.30 x 0.22 x 0.13 m @ 2.0 kg:
+           Ixx = m/12 * (y^2 + z^2) = 2/12 * (0.0484 + 0.0169) = 0.0109
+           Iyy = m/12 * (x^2 + z^2) = 2/12 * (0.09 + 0.0169) = 0.0178
+           Izz = m/12 * (x^2 + y^2) = 2/12 * (0.09 + 0.0484) = 0.0231 -->
+      <inertia
+        ixx="0.0109" ixy="0" ixz="0"
+        iyy="0.0178" iyz="0"
+        izz="0.0231"/>
     </inertial>
     <visual>
@@ -57,9 +69,9 @@
     </collision>
   </link>
-  <!-- Left wheel: positive y side -->
+  <!-- Left wheel: positive y side, FORWARD of chassis center (x = +0.05) -->
   <joint name="left_wheel_joint" type="continuous">
     <parent link="base_link"/>
     <child link="left_wheel"/>
-    <origin xyz="0 ${track/2} -${wheel_radius}" rpy="-1.5707 0 0"/>
+    <origin xyz="${wheel_offset_x} ${track/2} -${wheel_radius}" rpy="-1.5707 0 0"/>
     <axis xyz="0 0 1"/>
     <dynamics damping="0.1" friction="0.1"/>
@@ -69,8 +81,11 @@
       <origin xyz="0 0 0" rpy="0 0 0"/>
       <mass value="${wheel_mass}"/>
-      <inertia
-        ixx="0.145833" ixy="0" ixz="0"
-        iyy="0.145833" iyz="0"
-        izz="0.125"/>
+      <!-- Solid cylinder r=0.04, h=0.02, m=0.1:
+           Ixx = Iyy = m/12 * (3r^2 + h^2) = 0.1/12 * (0.0048 + 0.0004) = 0.0000433
+           Izz = m r^2 / 2 = 0.1 * 0.0016 / 2 = 0.00008 -->
+      <inertia
+        ixx="0.0000433" ixy="0" ixz="0"
+        iyy="0.0000433" iyz="0"
+        izz="0.00008"/>
     </inertial>
     <visual>
@@ -90,9 +105,9 @@
     </collision>
   </link>
-  <!-- Right wheel: negative y side -->
+  <!-- Right wheel: negative y side, FORWARD of chassis center (x = +0.05) -->
   <joint name="right_wheel_joint" type="continuous">
     <parent link="base_link"/>
     <child link="right_wheel"/>
-    <origin xyz="0 -${track/2} -${wheel_radius}" rpy="-1.5707 0 0"/>
+    <origin xyz="${wheel_offset_x} -${track/2} -${wheel_radius}" rpy="-1.5707 0 0"/>
     <axis xyz="0 0 1"/>
     <dynamics damping="0.1" friction="0.1"/>
@@ -103,7 +118,7 @@
       <mass value="${wheel_mass}"/>
       <inertia
-        ixx="0.145833" ixy="0" ixz="0"
-        iyy="0.145833" iyz="0"
-        izz="0.125"/>
+        ixx="0.0000433" ixy="0" ixz="0"
+        iyy="0.0000433" iyz="0"
+        izz="0.00008"/>
     </inertial>
     <visual>
@@ -123,23 +138,28 @@
     </collision>
   </link>
-  <!-- Caster ball (rear, passive) -->
+  <!-- Single rear caster ball (passive). Same offset z as the drive wheels
+       (-wheel_radius) so the caster sphere bottom rests on the ground at the
+       same plane as the wheel bottoms. Ball-jointed at the chassis for free
+       yaw. Layout matches visualize_lidar.sdf's vehicle_blue: 2 forward drive
+       wheels + 1 rear caster, forming a stable 3-point contact polygon. -->
   <joint name="caster_wheel_joint" type="fixed">
     <parent link="base_link"/>
-    <child link="caster"/>
+    <child link="caster_back"/>
     <origin xyz="${caster_offset_x} 0 -${wheel_radius}" rpy="0 0 0"/>
   </joint>
-  <link name="caster">
+  <link name="caster_back">
     <inertial>
       <origin xyz="0 0 0" rpy="0 0 0"/>
       <mass value="${caster_mass}"/>
-      <inertia
-        ixx="0.1" ixy="0" ixz="0"
-        iyy="0.1" iyz="0"
-        izz="0.1"/>
-    </inertial>
-    <visual>
-      <origin xyz="0 0 0" rpy="0 0 0"/>
-      <geometry>
-        <sphere radius="${caster_radius}"/>
+      <!-- Solid sphere r=0.04, m=0.05: I = 2/5 m r^2 = 0.4 * 0.05 * 0.0016 = 0.000032 -->
+      <inertia
+        ixx="0.000032" ixy="0" ixz="0"
+        iyy="0.000032" iyz="0"
+        izz="0.000032"/>
+    </inertial>
+    <visual>
+      <origin xyz="0 0 0" rpy="0 0 0"/>
+      <geometry>
+        <sphere radius="${wheel_radius}"/>
       </geometry>
       <material name="caster_dark">
@@ -150,5 +170,5 @@
       <origin xyz="0 0 0" rpy="0 0 0"/>
       <geometry>
-        <sphere radius="${caster_radius}"/>
+        <sphere radius="${wheel_radius}"/>
       </geometry>
     </collision>

Commit message: refactor: Update gz sim vehicle to use back wheels encoder

File: src/smb_robot/urdf/smb.urdf.xacro (robot description, xacro)
@@ -21,10 +21,10 @@
   <xacro:property name="wheel_thickness" value="0.02"/>
   <xacro:property name="track"          value="0.22"/>
-  <!-- Drive wheels forward of chassis center (x = +0.05), single caster at the
-       rear (x = -0.105). This mirrors the visualize_lidar.sdf reference layout:
-       wheels carry the front load, caster balances the rear. Masses/inertia
-       sized for a chibi ~30cm supermarket robot. -->
-  <xacro:property name="wheel_offset_x" value="0.05"/>
-  <xacro:property name="caster_offset_x" value="-0.105"/>
+  <!-- Drive wheels at the REAR of the chassis (x = -0.05), driven by motors with
+       encoders — matches the real robot layout. Single ball caster at the front
+       (x = +0.05) for free-rolling turns. Ball joint is critical: the front caster
+       must roll freely during rotation so DiffDrive odometry stays accurate. -->
+  <xacro:property name="wheel_offset_x" value="-0.05"/>
+  <xacro:property name="caster_offset_x" value="+0.05"/>
   <!-- Caster uses the same radius as the drive wheels so all three contact
        points lie on the same ground plane. The wheel_radius property above
@@ -69,5 +69,5 @@
     </collision>
   </link>
-  <!-- Left wheel: positive y side, FORWARD of chassis center (x = +0.05) -->
+  <!-- Left rear drive wheel: positive y side, REAR of chassis -->
   <joint name="left_wheel_joint" type="continuous">
     <parent link="base_link"/>
@@ -105,5 +105,5 @@
     </collision>
   </link>
-  <!-- Right wheel: negative y side, FORWARD of chassis center (x = +0.05) -->
+  <!-- Right rear drive wheel: negative y side, REAR of chassis -->
   <joint name="right_wheel_joint" type="continuous">
     <parent link="base_link"/>
@@ -138,15 +138,15 @@
     </collision>
   </link>
-  <!-- Single rear caster ball (passive). Same offset z as the drive wheels
+  <!-- One passive front ball caster (free-rolling). Same offset z as the drive wheels
        (-wheel_radius) so the caster sphere bottom rests on the ground at the
-       same plane as the wheel bottoms. Ball-jointed at the chassis for free
-       yaw. Layout matches visualize_lidar.sdf's vehicle_blue: 2 forward drive
-       wheels + 1 rear caster, forming a stable 3-point contact polygon. -->
-  <joint name="caster_wheel_joint" type="fixed">
-    <parent link="base_link"/>
-    <child link="caster_back"/>
+       same plane as the wheel bottoms.
+       URDF uses 'fixed' (KDL/RViz limitation; ball is SDF-only).
+       SDF uses 'ball' for Gazebo free-rolling physics. -->
+  <joint name="caster_front_joint" type="fixed">
+    <parent link="base_link"/>
+    <child link="caster_front"/>
     <origin xyz="${caster_offset_x} 0 -${wheel_radius}" rpy="0 0 0"/>
   </joint>
-  <link name="caster_back">
+  <link name="caster_front">
     <inertial>
       <origin xyz="0 0 0" rpy="0 0 0"/>

Commit message: fix: Fix SLAM-odom out of sync problem

File: src/smb_robot/urdf/smb.urdf.xacro (robot description, xacro)
@@ -176,13 +176,14 @@
     </collision>
   </link>
-  <!-- Laser frame: mounted on the LEFT side of chassis (x = -0.05, y = 0),
-       with -90° yaw so lidar angle_min=0 points along URDF +Y = physical forward (wall).
-       Scan data: wall at ~315-340° = URDF +Y direction. ESP32 publishes angle 0°
-       in the chassis +Y direction, so rpy=0 0 -1.5708 makes lidar +X align with chassis +Y. -->
+  <!-- Laser frame: mounted on the LEFT side of chassis (x = -0.05).
+       LiDAR angle_min=0° points along URDF +X = physical forward.
+       No extra rotation: YDLidar X3 angle 0° is already in the forward direction.
+       ESP32 publishes scan with frame_id="laser_frame"; robot_state_publisher
+       provides the TF map → odom → base_link → laser_frame. -->
   <xacro:property name="lidar_offset_x" value="-0.05"/>
   <joint name="lidar_joint" type="fixed">
     <parent link="base_link"/>
     <child link="laser_frame"/>
-    <origin xyz="${lidar_offset_x} 0 ${lidar_offset_z}" rpy="0 0 -1.5707"/>
+    <origin xyz="${lidar_offset_x} 0 ${lidar_offset_z}" rpy="0 0 0"/>
   </joint>
   <link name="laser_frame">

Commit message: fix: Fix urdf orientation + fix basic nav2 logic

File: src/smb_robot/urdf/smb.urdf.xacro (robot description, xacro)
@@ -185,5 +185,5 @@
     <parent link="base_link"/>
     <child link="laser_frame"/>
-    <origin xyz="${lidar_offset_x} 0 ${lidar_offset_z}" rpy="0 0 0"/>
+    <origin xyz="${lidar_offset_x} 0 ${lidar_offset_z}" rpy="0 0 -1.5707"/>
   </joint>
   <link name="laser_frame">

Commit message: Fix LiDAR timestamps, remove future-stamping from Odometry relay, and configure SLAM Toolbox

File: src/smb_robot/urdf/smb.urdf.xacro (robot description, xacro)
@@ -176,10 +176,10 @@
     </collision>
   </link>
-  <!-- Laser frame: mounted on the LEFT side of chassis (x = -0.05).
+  <!-- Laser frame: center-mounted on chassis (x = 0.0) and connected directly to Pi 5 USB (not through ESP32).
        LiDAR angle_min=0° points along URDF +X = physical forward.
        No extra rotation: YDLidar X3 angle 0° is already in the forward direction.
-       ESP32 publishes scan with frame_id="laser_frame"; robot_state_publisher
+       Driver publishes scan with frame_id="laser_frame"; robot_state_publisher
        provides the TF map → odom → base_link → laser_frame. -->
-  <xacro:property name="lidar_offset_x" value="-0.05"/>
+  <xacro:property name="lidar_offset_x" value="0.0"/>
   <joint name="lidar_joint" type="fixed">
     <parent link="base_link"/>

Commit message: fix: Fix lidar urdf direction

File: src/smb_robot/urdf/smb.urdf.xacro (robot description, xacro)
@@ -27,6 +27,6 @@
        Scan data: lidar on back (-X) with 180° rotation so angle 0° faces backward
        (toward wall = physical front). -->
-  <xacro:property name="wheel_offset_x" value="0.05"/>
-  <xacro:property name="caster_offset_x" value="-0.05"/>
+  <xacro:property name="wheel_offset_x" value="-0.05"/>
+  <xacro:property name="caster_offset_x" value="0.05"/>
   <!-- Caster uses the same radius as the drive wheels so all three contact
        points lie on the same ground plane. The wheel_radius property above
@@ -185,5 +185,5 @@
     <parent link="base_link"/>
     <child link="laser_frame"/>
-    <origin xyz="${lidar_offset_x} 0 ${lidar_offset_z}" rpy="0 0 -1.5707"/>
+    <origin xyz="${lidar_offset_x} 0 ${lidar_offset_z}" rpy="0 0 1.5708"/>
   </joint>
   <link name="laser_frame">

Commit message: fix: Fix rviz orientation problem

File: src/smb_robot/urdf/smb.urdf.xacro (robot description, xacro)
@@ -185,5 +185,5 @@
     <parent link="base_link"/>
     <child link="laser_frame"/>
-    <origin xyz="${lidar_offset_x} 0 ${lidar_offset_z}" rpy="0 0 1.5708"/>
+    <origin xyz="${lidar_offset_x} 0 ${lidar_offset_z}" rpy="0 0 -1.5708"/>
   </joint>
   <link name="laser_frame">

Commit message: refactor: Refactor urdf + supersonic logic

File: src/smb_robot/urdf/smb.urdf.xacro (robot description, xacro)
@@ -15,7 +15,7 @@
 -->
 <robot xmlns:xacro="http://www.ros.org/wiki/xacro" name="smb">
-  <xacro:property name="chassis_length" value="0.30"/>
-  <xacro:property name="chassis_width"  value="0.22"/>
-  <xacro:property name="chassis_height" value="0.13"/>
+  <xacro:property name="chassis_length" value="0.27"/>
+  <xacro:property name="chassis_width"  value="0.145"/>
+  <xacro:property name="chassis_height" value="0.075"/>
   <xacro:property name="wheel_radius"   value="0.04"/>
   <xacro:property name="wheel_thickness" value="0.02"/>
@@ -32,5 +32,5 @@
        points lie on the same ground plane. The wheel_radius property above
        is reused for the caster sphere. -->
-  <xacro:property name="lidar_offset_z" value="0.075"/>
+  <xacro:property name="lidar_offset_z" value="0.36"/>
   <xacro:property name="imu_offset_z"   value="0.05"/>
   <!-- Masses kept low so the sim runs smoothly; chassis dominates the dynamics. -->
@@ -237,3 +237,32 @@
     </collision>
   </link>
+  <!-- Ultrasonic Sensors -->
+  <!-- Front -->
+  <joint name="us_front_joint" type="fixed">
+    <parent link="base_link"/>
+    <child link="us_front_link"/>
+    <origin xyz="0.135 0 0" rpy="0 0 0"/>
+  </joint>
+  <link name="us_front_link"/>
+  <!-- Rear -->
+  <joint name="us_rear_joint" type="fixed">
+    <parent link="base_link"/>
+    <child link="us_rear_link"/>
+    <origin xyz="-0.135 0 0" rpy="0 0 3.14159"/>
+  </joint>
+  <link name="us_rear_link"/>
+  <!-- Left -->
+  <joint name="us_left_joint" type="fixed">
+    <parent link="base_link"/>
+    <child link="us_left_link"/>
+    <origin xyz="0 0.0725 0" rpy="0 0 1.5708"/>
+  </joint>
+  <link name="us_left_link"/>
+  <!-- Right -->
+  <joint name="us_right_joint" type="fixed">
+    <parent link="base_link"/>
+    <child link="us_right_link"/>
+    <origin xyz="0 -0.0725 0" rpy="0 0 -1.5708"/>
+  </joint>
+  <link name="us_right_link"/>
 </robot>

Commit message: update: Update FE-ROS2 bridge

File: src/smb_robot/urdf/smb.urdf.xacro (robot description, xacro)
@@ -44,5 +44,5 @@
          with no dynamics). The dummy chassis makes KDL happy. -->
     <inertial>
-      <origin xyz="0 0 0" rpy="0 0 0"/>
+      <origin xyz="0 0 0" rpy="0 0 -1.5708"/>
       <mass value="${chassis_mass}"/>
       <!-- Box inertia for 0.30 x 0.22 x 0.13 m @ 2.0 kg:
@@ -56,5 +56,5 @@
     </inertial>
     <visual>
-      <origin xyz="0 0 0" rpy="0 0 0"/>
+      <origin xyz="0 0 0" rpy="0 0 -1.5708"/>
       <geometry>
         <box size="${chassis_length} ${chassis_width} ${chassis_height}"/>
@@ -65,5 +65,5 @@
     </visual>
     <collision>
-      <origin xyz="0 0 0" rpy="0 0 0"/>
+      <origin xyz="0 0 0" rpy="0 0 -1.5708"/>
       <geometry>
         <box size="${chassis_length} ${chassis_width} ${chassis_height}"/>
@@ -81,5 +81,5 @@
   <link name="left_wheel">
     <inertial>
-      <origin xyz="0 0 0" rpy="0 0 0"/>
+      <origin xyz="0 0 0" rpy="0 0 -1.5708"/>
       <mass value="${wheel_mass}"/>
       <!-- Solid cylinder r=0.04, h=0.02, m=0.1:
@@ -92,5 +92,5 @@
     </inertial>
     <visual>
-      <origin xyz="0 0 0" rpy="0 0 0"/>
+      <origin xyz="0 0 0" rpy="0 0 -1.5708"/>
       <geometry>
         <cylinder radius="${wheel_radius}" length="${wheel_thickness}"/>
@@ -101,5 +101,5 @@
     </visual>
     <collision>
-      <origin xyz="0 0 0" rpy="0 0 0"/>
+      <origin xyz="0 0 0" rpy="0 0 -1.5708"/>
       <geometry>
         <cylinder radius="${wheel_radius}" length="${wheel_thickness}"/>
@@ -117,5 +117,5 @@
   <link name="right_wheel">
     <inertial>
-      <origin xyz="0 0 0" rpy="0 0 0"/>
+      <origin xyz="0 0 0" rpy="0 0 -1.5708"/>
       <mass value="${wheel_mass}"/>
       <inertia
@@ -125,5 +125,5 @@
     </inertial>
     <visual>
-      <origin xyz="0 0 0" rpy="0 0 0"/>
+      <origin xyz="0 0 0" rpy="0 0 -1.5708"/>
       <geometry>
         <cylinder radius="${wheel_radius}" length="${wheel_thickness}"/>
@@ -134,5 +134,5 @@
     </visual>
     <collision>
-      <origin xyz="0 0 0" rpy="0 0 0"/>
+      <origin xyz="0 0 0" rpy="0 0 -1.5708"/>
       <geometry>
         <cylinder radius="${wheel_radius}" length="${wheel_thickness}"/>
@@ -148,9 +148,9 @@
     <parent link="base_link"/>
     <child link="caster_front"/>
-    <origin xyz="${caster_offset_x} 0 -${wheel_radius}" rpy="0 0 0"/>
+    <origin xyz="${caster_offset_x} 0 -${wheel_radius}" rpy="0 0 -1.5708"/>
   </joint>
   <link name="caster_front">
     <inertial>
-      <origin xyz="0 0 0" rpy="0 0 0"/>
+      <origin xyz="0 0 0" rpy="0 0 -1.5708"/>
       <mass value="${caster_mass}"/>
       <!-- Solid sphere r=0.04, m=0.05: I = 2/5 m r^2 = 0.4 * 0.05 * 0.0016 = 0.000032 -->
@@ -161,5 +161,5 @@
     </inertial>
     <visual>
-      <origin xyz="0 0 0" rpy="0 0 0"/>
+      <origin xyz="0 0 0" rpy="0 0 -1.5708"/>
       <geometry>
         <sphere radius="${wheel_radius}"/>
@@ -170,5 +170,5 @@
     </visual>
     <collision>
-      <origin xyz="0 0 0" rpy="0 0 0"/>
+      <origin xyz="0 0 0" rpy="0 0 -1.5708"/>
       <geometry>
         <sphere radius="${wheel_radius}"/>
@@ -189,10 +189,10 @@
   <link name="laser_frame">
     <inertial>
-      <origin xyz="0 0 0" rpy="0 0 0"/>
+      <origin xyz="0 0 0" rpy="0 0 -1.5708"/>
       <mass value="0.1"/>
       <inertia ixx="0.001" ixy="0" ixz="0" iyy="0.001" iyz="0" izz="0.001"/>
     </inertial>
     <visual>
-      <origin xyz="0 0 0" rpy="0 0 0"/>
+      <origin xyz="0 0 0" rpy="0 0 -1.5708"/>
       <geometry>
         <cylinder radius="0.025" length="0.025"/>
@@ -203,5 +203,5 @@
     </visual>
     <collision>
-      <origin xyz="0 0 0" rpy="0 0 0"/>
+      <origin xyz="0 0 0" rpy="0 0 -1.5708"/>
       <geometry>
         <cylinder radius="0.025" length="0.025"/>
@@ -213,14 +213,14 @@
     <parent link="base_link"/>
     <child link="imu_link"/>
-    <origin xyz="0 0 ${imu_offset_z}" rpy="0 0 0"/>
+    <origin xyz="0 0 ${imu_offset_z}" rpy="0 0 -1.5708"/>
   </joint>
   <link name="imu_link">
     <inertial>
-      <origin xyz="0 0 0" rpy="0 0 0"/>
+      <origin xyz="0 0 0" rpy="0 0 -1.5708"/>
       <mass value="0.01"/>
       <inertia ixx="0.0001" ixy="0" ixz="0" iyy="0.0001" iyz="0" izz="0.0001"/>
     </inertial>
     <visual>
-      <origin xyz="0 0 0" rpy="0 0 0"/>
+      <origin xyz="0 0 0" rpy="0 0 -1.5708"/>
       <geometry>
         <box size="0.02 0.02 0.005"/>
@@ -231,5 +231,5 @@
     </visual>
     <collision>
-      <origin xyz="0 0 0" rpy="0 0 0"/>
+      <origin xyz="0 0 0" rpy="0 0 -1.5708"/>
       <geometry>
         <box size="0.02 0.02 0.005"/>
@@ -242,5 +242,5 @@
     <parent link="base_link"/>
     <child link="us_front_link"/>
-    <origin xyz="0.135 0 0" rpy="0 0 0"/>
+    <origin xyz="0.135 0 0" rpy="0 0 -1.5708"/>
   </joint>
   <link name="us_front_link"/>

Commit message: feat: Add interactive Map Editor endpoint and AI Camera integration

File: src/smb_robot/urdf/smb.urdf.xacro (robot description, xacro)
@@ -266,3 +266,34 @@
   </joint>
   <link name="us_right_link"/>
+  <!-- AI Camera IMX500 -->
+  <joint name="camera_joint" type="fixed">
+    <parent link="base_link"/>
+    <child link="camera_link"/>
+    <!-- Positioned at the front of the robot, facing forward (URDF +X) -->
+    <!-- Note: Actual offsets (xyz) depend on physical mounting,
+         using placeholder values (x: front edge, z: above chassis) -->
+    <origin xyz="0.135 0 0.15" rpy="0 0 0"/>
+  </joint>
+  <link name="camera_link">
+    <inertial>
+      <origin xyz="0 0 0" rpy="0 0 0"/>
+      <mass value="0.05"/>
+      <inertia ixx="0.0001" ixy="0" ixz="0" iyy="0.0001" iyz="0" izz="0.0001"/>
+    </inertial>
+    <visual>
+      <origin xyz="0 0 0" rpy="0 0 0"/>
+      <geometry>
+        <box size="0.02 0.04 0.02"/>
+      </geometry>
+      <material name="camera_black">
+        <color rgba="0.1 0.1 0.1 1"/>
+      </material>
+    </visual>
+    <collision>
+      <origin xyz="0 0 0" rpy="0 0 0"/>
+      <geometry>
+        <box size="0.02 0.04 0.02"/>
+      </geometry>
+    </collision>
+  </link>
 </robot>
